File: board_control.kicad_sch (KiCad schematic)
At the start: 40 parts, among them J4 Conn_01x09_Pin

Commit message: Mounting holes positioned, and routing
Parts:
- added H1 (x4): Board MountingHole, MountingHole:MountingHole_2.7mm_M2.5_Pad_Via, symbol Mechanical:MountingHole
- added J10: Conn_01x02_Pin, Connector_PinHeader_2.54mm:PinHeader_1x02_P2.54mm_Vertical, symbol Connector:Conn_01x02_Pin
- H1: footprint MountingHole:MountingHole_4.3mm_M4_Pad_Via -> MountingHole:MountingHole_2.7mm_M2.5_Pad_Via
Connections:
- net VCCOUT: now also J10.2 (Pin_2)
- net at D5.1 (K), R23.2: now also J10.1 (Pin_1)
Changed lines of the file:
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@@
   (junction (at 114.3 40.64) (diameter 0) (color 0 0 0 0)
   )
+  (junction (at 267.97 29.21) (diameter 0) (color 0 0 0 0)
+  )
   (junction (at 153.67 30.48) (diameter 0) (color 0 0 0 0)
   )
@@
   (junction (at 55.88 39.37) (diameter 0) (color 0 0 0 0)
   )
+  (junction (at 267.97 41.91) (diameter 0) (color 0 0 0 0)
+  )
   (junction (at 48.26 124.46) (diameter 0) (color 0 0 0 0)
   )
@@
     (stroke (width 0) (type default))
   )
+  (wire (pts (xy 276.86 39.37) (xy 276.86 41.91))
+    (stroke (width 0) (type default))
+  )
   (wire (pts (xy 111.76 50.8) (xy 127 50.8))
     (stroke (width 0) (type default))
   )
+  (wire (pts (xy 276.86 36.83) (xy 276.86 29.21))
+    (stroke (width 0) (type default))
+  )
   (wire (pts (xy 81.28 40.64) (xy 81.28 36.83))
     (stroke (width 0) (type default))
@@
     (stroke (width 0) (type default))
   )
+  (wire (pts (xy 276.86 41.91) (xy 267.97 41.91))
+    (stroke (width 0) (type default))
+  )
   (wire (pts (xy 165.1 31.75) (xy 165.1 30.48))
     (stroke (width 0) (type default))
@@
   )
   (wire (pts (xy 149.86 93.98) (xy 172.72 93.98))
+    (stroke (width 0) (type default))
+  )
+  (wire (pts (xy 276.86 29.21) (xy 267.97 29.21))
     (stroke (width 0) (type default))
   )
@@
     )
   )
+  (symbol (lib_id "Mechanical:MountingHole") (at 265.43 147.32 0) (unit 1)
+    (in_bom yes) (on_board yes) (dnp no) (fields_autoplaced)
+    (property "Reference" "H1" (at 267.97 146.05 0)
+      (effects (font (size 1.27 1.27)) (justify left))
+    )
+    (property "Value" "Board MountingHole" (at 267.97 148.59 0)
+      (effects (font (size 1.27 1.27)) (justify left))
+    )
+    (property "Footprint" "MountingHole:MountingHole_2.7mm_M2.5_Pad_Via" (at 265.43 147.32 0)
+      (effects (font (size 1.27 1.27)) hide)
+    )
+    (property "Datasheet" "~" (at 265.43 147.32 0)
+      (effects (font (size 1.27 1.27)) hide)
+    )
+    (instances
+      (project "jumpstarter"
+        (path "/5e49fb74-0a9b-4946-8b59-2b8244d10fd9"
+          (reference "H1") (unit 1)
+        )
+        (path "/5e49fb74-0a9b-4946-8b59-2b8244d10fd9/0a246f5a-dd08-4f47-947a-3b89ae06d789"
+          (reference "H15") (unit 1)
+        )
+      )
+    )
+  )
   (symbol (lib_id "power:GND") (at 134.62 66.04 0) (unit 1)
     (in_bom yes) (on_board yes) (dnp no) (fields_autoplaced)
@@
         (path "/5e49fb74-0a9b-4946-8b59-2b8244d10fd9/0a246f5a-dd08-4f47-947a-3b89ae06d789"
           (reference "C12") (unit 1)
+        )
+      )
+    )
+  )
+  (symbol (lib_id "Connector:Conn_01x02_Pin") (at 281.94 39.37 180) (unit 1)
+    (in_bom yes) (on_board yes) (dnp no) (fields_autoplaced)
+    (property "Reference" "J10" (at 283.21 38.1 0)
+      (effects (font (size 1.27 1.27)) (justify right))
+    )
+    (property "Value" "Conn_01x02_Pin" (at 283.21 39.37 0)
+      (effects (font (size 1.27 1.27)) (justify right) hide)
+    )
+    (property "Footprint" "Connector_PinHeader_2.54mm:PinHeader_1x02_P2.54mm_Vertical" (at 281.94 39.37 0)
+      (effects (font (size 1.27 1.27)) hide)
+    )
+    (property "Datasheet" "~" (at 281.94 39.37 0)
+      (effects (font (size 1.27 1.27)) hide)
+    )
+    (pin "1")
+    (pin "2")
+    (instances
+      (project "jumpstarter"
+        (path "/5e49fb74-0a9b-4946-8b59-2b8244d10fd9"
+          (reference "J10") (unit 1)
+        )
+        (path "/5e49fb74-0a9b-4946-8b59-2b8244d10fd9/0a246f5a-dd08-4f47-947a-3b89ae06d789"
+          (reference "J16") (unit 1)
         )
       )
@@
       (effects (font (size 1.27 1.27)) (justify left))
     )
-    (property "Footprint" "MountingHole:MountingHole_4.3mm_M4_Pad_Via" (at 172.72 153.67 0)
+    (property "Footprint" "MountingHole:MountingHole_2.7mm_M2.5_Pad_Via" (at 172.72 153.67 0)
       (effects (font (size 1.27 1.27)) hide)
     )
@@
       (effects (font (size 1.27 1.27)) (justify left))
     )
-    (property "Footprint" "MountingHole:MountingHole_4.3mm_M4_Pad_Via" (at 172.72 134.62 0)
+    (property "Footprint" "MountingHole:MountingHole_2.7mm_M2.5_Pad_Via" (at 172.72 134.62 0)
       (effects (font (size 1.27 1.27)) hide)
     )
@@
       (effects (font (size 1.27 1.27)) (justify left))
     )
-    (property "Footprint" "MountingHole:MountingHole_4.3mm_M4_Pad_Via" (at 204.47 134.62 0)
+    (property "Footprint" "MountingHole:MountingHole_2.7mm_M2.5_Pad_Via" (at 204.47 134.62 0)
       (effects (font (size 1.27 1.27)) hide)
     )
@@
         (path "/5e49fb74-0a9b-4946-8b59-2b8244d10fd9/0a246f5a-dd08-4f47-947a-3b89ae06d789"
           (reference "#PWR042") (unit 1)
+        )
+      )
+    )
+  )
+  (symbol (lib_id "Mechanical:MountingHole") (at 233.68 153.67 0) (unit 1)
+    (in_bom yes) (on_board yes) (dnp no) (fields_autoplaced)
+    (property "Reference" "H1" (at 236.22 152.4 0)
+      (effects (font (size 1.27 1.27)) (justify left))
+    )
+    (property "Value" "Board MountingHole" (at 236.22 154.94 0)
+      (effects (font (size 1.27 1.27)) (justify left))
+    )
+    (property "Footprint" "MountingHole:MountingHole_2.7mm_M2.5_Pad_Via" (at 233.68 153.67 0)
+      (effects (font (size 1.27 1.27)) hide)
+    )
+    (property "Datasheet" "~" (at 233.68 153.67 0)
+      (effects (font (size 1.27 1.27)) hide)
+    )
+    (instances
+      (project "jumpstarter"
+        (path "/5e49fb74-0a9b-4946-8b59-2b8244d10fd9"
+          (reference "H1") (unit 1)
+        )
+        (path "/5e49fb74-0a9b-4946-8b59-2b8244d10fd9/0a246f5a-dd08-4f47-947a-3b89ae06d789"
+          (reference "H14") (unit 1)
         )
       )
@@
       (effects (font (size 1.27 1.27)) (justify left))
     )
-    (property "Footprint" "MountingHole:MountingHole_4.3mm_M4_Pad_Via" (at 172.72 140.97 0)
+    (property "Footprint" "MountingHole:MountingHole_2.7mm_M2.5_Pad_Via" (at 172.72 140.97 0)
       (effects (font (size 1.27 1.27)) hide)
     )
@@
       (effects (font (size 1.27 1.27)) (justify left))
     )
-    (property "Footprint" "MountingHole:MountingHole_4.3mm_M4_Pad_Via" (at 204.47 147.32 0)
+    (property "Footprint" "MountingHole:MountingHole_2.7mm_M2.5_Pad_Via" (at 204.47 147.32 0)
       (effects (font (size 1.27 1.27)) hide)
     )
@@
         (path "/5e49fb74-0a9b-4946-8b59-2b8244d10fd9/0a246f5a-dd08-4f47-947a-3b89ae06d789"
           (reference "H10") (unit 1)
+        )
+      )
+    )
+  )
+  (symbol (lib_id "Mechanical:MountingHole") (at 233.68 147.32 0) (unit 1)
+    (in_bom yes) (on_board yes) (dnp no) (fields_autoplaced)
+    (property "Reference" "H1" (at 236.22 146.05 0)
+      (effects (font (size 1.27 1.27)) (justify left))
+    )
+    (property "Value" "Board MountingHole" (at 236.22 148.59 0)
+      (effects (font (size 1.27 1.27)) (justify left))
+    )
+    (property "Footprint" "MountingHole:MountingHole_2.7mm_M2.5_Pad_Via" (at 233.68 147.32 0)
+      (effects (font (size 1.27 1.27)) hide)
+    )
+    (property "Datasheet" "~" (at 233.68 147.32 0)
+      (effects (font (size 1.27 1.27)) hide)
+    )
+    (instances
+      (project "jumpstarter"
+        (path "/5e49fb74-0a9b-4946-8b59-2b8244d10fd9"
+          (reference "H1") (unit 1)
+        )
+        (path "/5e49fb74-0a9b-4946-8b59-2b8244d10fd9/0a246f5a-dd08-4f47-947a-3b89ae06d789"
+          (reference "H13") (unit 1)
         )
       )
@@
       (effects (font (size 1.27 1.27)) (justify left))
     )
-    (property "Footprint" "MountingHole:MountingHole_4.3mm_M4_Pad_Via" (at 204.47 140.97 0)
+    (property "Footprint" "MountingHole:MountingHole_2.7mm_M2.5_Pad_Via" (at 204.47 140.97 0)
       (effects (font (size 1.27 1.27)) hide)
     )
@@
       (effects (font (size 1.27 1.27)) (justify left))
     )
-    (property "Footprint" "MountingHole:MountingHole_4.3mm_M4_Pad_Via" (at 204.47 153.67 0)
+    (property "Footprint" "MountingHole:MountingHole_2.7mm_M2.5_Pad_Via" (at 204.47 153.67 0)
       (effects (font (size 1.27 1.27)) hide)
     )
@@
         (path "/5e49fb74-0a9b-4946-8b59-2b8244d10fd9/0a246f5a-dd08-4f47-947a-3b89ae06d789"
           (reference "#PWR062") (unit 1)
+        )
+      )
+    )
+  )
+  (symbol (lib_id "Mechanical:MountingHole") (at 265.43 153.67 0) (unit 1)
+    (in_bom yes) (on_board yes) (dnp no) (fields_autoplaced)
+    (property "Reference" "H1" (at 267.97 152.4 0)
+      (effects (font (size 1.27 1.27)) (justify left))
+    )
+    (property "Value" "Board MountingHole" (at 267.97 154.94 0)
+      (effects (font (size 1.27 1.27)) (justify left))
+    )
+    (property "Footprint" "MountingHole:MountingHole_2.7mm_M2.5_Pad_Via" (at 265.43 153.67 0)
+      (effects (font (size 1.27 1.27)) hide)
+    )
+    (property "Datasheet" "~" (at 265.43 153.67 0)
+      (effects (font (size 1.27 1.27)) hide)
+    )
+    (instances
+      (project "jumpstarter"
+        (path "/5e49fb74-0a9b-4946-8b59-2b8244d10fd9"
+          (reference "H1") (unit 1)
+        )
+        (path "/5e49fb74-0a9b-4946-8b59-2b8244d10fd9/0a246f5a-dd08-4f47-947a-3b89ae06d789"
+          (reference "H16") (unit 1)
         )
       )
@@
       (effects (font (size 1.27 1.27)) (justify left))
     )
-    (property "Footprint" "MountingHole:MountingHole_4.3mm_M4_Pad_Via" (at 172.72 147.32 0)
-      (effects (font (size 1.27 1.27)) hide)
-    )
+    (property "Footprint" "MountingHole:MountingHole_2.7mm_M2.5_Pad_Via" (at 172.72 147.32 0)
+      (effects (font (size 1.27 1.27)) hide)
+    )

Commit message: Update
Parts:
- added C15: 1nF, Capacitor_SMD:C_0603_1608Metric_Pad1.08x0.95mm_HandSolder, symbol Device:C
- added C?: 1uF, Capacitor_SMD:C_0603_1608Metric_Pad1.08x0.95mm_HandSolder, symbol Device:C
- U?: value ACS722xLCTR-20AU -> ACS725LLCTR-05AB-T
Connections:
- net GND: now also H1.1, H1.1, H1.1, H1.1, H1.1, H1.1, H1.1, H1.1, H1.1, H1.1, H1.1, H1.1, C?.1
- net GNDA: now also C15.2
- net VCCOUT: now also U?.1 (IP+), U?.2 (IP+); no longer U?.3 (IP-), U?.4 (IP-)
- net VCCOUT_SW: now also U?.3 (IP-), U?.4 (IP-); no longer U?.1 (IP+), U?.2 (IP+)
- net CURRENT_BWSEL: no longer names the net of U?.6 (BW_SEL)
- net CURRENT_BWSEL: now also C15.1
- net V_IO renamed +3.3V
- net +3.3V: now also C?.2
