File: jumpstarter.kicad_sch (KiCad schematic)
At the start: 65 parts, among them J10 Conn_01x02_Pin, J11 Conn_01x02_Pin, J12 Conn_01x02_Pin, J13 Conn_01x02_Pin, J14 Conn_01x02_Pin, J15 Conn_01x02_Pin, J6 Conn_01x05_Pin, P1 USB_C_Plug_USB2.0, SW1 SW_Push, SW2 SW_Push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

Commit message: Mounting holes positioned, and routing
Parts:
- added H17, H18: ITX MountingHole, MountingHole:MountingHole_4.3mm_M4_Pad_Via, symbol Mechanical:MountingHole
Changed lines of the file:
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@@
+    )
+  )
+  (symbol (lib_id "Mechanical:MountingHole") (at 209.55 15.24 0) (unit 1)
+    (in_bom yes) (on_board yes) (dnp no) (fields_autoplaced)
+    (property "Reference" "H17" (at 212.09 13.97 0)
+      (effects (font (size 1.27 1.27)) (justify left))
+    )
+    (property "Value" "ITX MountingHole" (at 212.09 16.51 0)
+      (effects (font (size 1.27 1.27)) (justify left))
+    )
+    (property "Footprint" "MountingHole:MountingHole_4.3mm_M4_Pad_Via" (at 209.55 15.24 0)
+      (effects (font (size 1.27 1.27)) hide)
+    )
+    (property "Datasheet" "~" (at 209.55 15.24 0)
+      (effects (font (size 1.27 1.27)) hide)
+    )
+    (instances
+      (project "jumpstarter"
+        (path "/5e49fb74-0a9b-4946-8b59-2b8244d10fd9"
+          (reference "H17") (unit 1)
+        )
+      )
     )
   )
@@
         )
       )
+    )
+  )
+  (symbol (lib_id "Mechanical:MountingHole") (at 238.76 15.24 0) (unit 1)
+    (in_bom yes) (on_board yes) (dnp no) (fields_autoplaced)
+    (property "Reference" "H18" (at 241.3 13.97 0)
+      (effects (font (size 1.27 1.27)) (justify left))
+    )
+    (property "Value" "ITX MountingHole" (at 241.3 16.51 0)
+      (effects (font (size 1.27 1.27)) (justify left))
+    )
+    (property "Footprint" "MountingHole:MountingHole_4.3mm_M4_Pad_Via" (at 238.76 15.24 0)
+      (effects (font (size 1.27 1.27)) hide)
+    )
+    (property "Datasheet" "~" (at 238.76 15.24 0)
+      (effects (font (size 1.27 1.27)) hide)
+    )
+    (instances
+      (project "jumpstarter"
+        (path "/5e49fb74-0a9b-4946-8b59-2b8244d10fd9"
+          (reference "H18") (unit 1)
+        )
+      )

Commit message: Update
Parts:
- removed TP8: TestPoint, TestPoint:TestPoint_Pad_D1.0mm, symbol Connector:TestPoint
- H17, H18: value ITX MountingHole -> cable strap hole
- J15: footprint (none) -> Connector_PinHeader_2.54mm:PinHeader_1x02_P2.54mm_Vertical
- SW1: footprint Button_Switch_SMD:SW_SPST_B3S-1000 -> Button_Switch_THT:SW_Tactile_SPST_Angled_PTS645Vx58-2LFS
- Y2: footprint Oscillator:Oscillator_SMD_EuroQuartz_XO53-4Pin_5.0x3.2mm -> Oscillator:Oscillator_SMD_EuroQuartz_XO32-4Pin_3.2x2.5mm
Connections:
- net GND: now also H1.1, H17.1, H18.1, H2.1, H3.1, H4.1
- net NRST: now also J6.5 (Pin_5)
- net BW_SEL: no longer names the net of U1.13 (PA3)
Other:
- sheet board_control ports: added none; removed CURRENT_BWSEL
